File: kicad/wii-breakout.sch (KiCad schematic (older format))
At the start: 9 parts, among them J1 Data Header, J2 USB Pads, J3 Bluetooth Pads, J4 GameCube Pads, J5 Reset Pad, J6 Audio Header, J7 Video Header, J8 Audio Pads, J9 Video Pads

Commit message: v1.0
Parts:
- added H1, H2: MountingHole_Pad, MountingHole:MountingHole_2.7mm_M2.5_Pad_Via, symbol Mechanical:MountingHole_Pad
- J1: value Data Header -> Peripherals
- J2: renamed from J6; value Audio Header -> Audio; footprint Connector_JST:JST_SH_BM02B-SRSS-TB_1x02-1MP_P1.00mm_Vertical -> Connector_JST:JST_SH_BM03B-SRSS-TB_1x03-1MP_P1.00mm_Vertical; symbol Connector_Generic_MountingPin:Conn_01x02_MountingPin -> Connector_Generic_MountingPin:Conn_01x03_MountingPin
- J3: renamed from J7; value Video Header -> Video; footprint Connector_JST:JST_SH_BM03B-SRSS-TB_1x03-1MP_P1.00mm_Vertical -> Connector_JST:JST_SH_BM04B-SRSS-TB_1x04-1MP_P1.00mm_Vertical; symbol Connector_Generic_MountingPin:Conn_01x03_MountingPin -> Connector_Generic_MountingPin:Conn_01x04_MountingPin
- J4: renamed from J2; value USB Pads -> USB
- J5: renamed from J4; value GameCube Pads -> GameCube
- J6: renamed from J5; value Reset Pad -> Reset
- J7: renamed from J3; value Bluetooth Pads -> Bluetooth
- J8: value Audio Pads -> Audio; footprint TestPoint:TestPoint_2Pads_2.0x1.0mm -> TestPoint:TestPoint_3Pads_2.0x1.0mm; symbol Connector:Conn_01x02_Male -> Connector:Conn_01x03_Male
- J9: value Video Pads -> Video; footprint TestPoint:TestPoint_3Pads_2.0x1.0mm -> TestPoint:TestPoint_4Pads_2.0x1.0mm; symbol Connector:Conn_01x03_Male -> Connector:Conn_01x04_Male
Connections:
- new net AUDIO_GND: J2.3 (Pin_3), J8.3 (Pin_3)
- new net GND: H1.1, H2.1
- new net VIDEO_GND: J3.4 (Pin_4), J9.4 (Pin_4)
- no-connect marks 0 -> 3
Changed lines of the file:
@@
 $EndDescr
 $Comp
-L Connector:Conn_01x02_Male J3
+L Connector:Conn_01x02_Male J7
 U 1 1 5E6B1D90
 P 3550 2450
-F 0 "J3" H 3522 2424 50  0000 R CNN
-F 1 "Bluetooth Pads" H 3522 2333 50  0000 R CNN
+F 0 "J7" H 3522 2424 50  0000 R CNN
+F 1 "Bluetooth" H 3522 2333 50  0000 R CNN
 F 2 "TestPoint:TestPoint_2Pads_2.0x1.0mm" H 3550 2450 50  0001 C CNN
 F 3 "~" H 3550 2450 50  0001 C CNN
@@
 	2800 1250 3350 1250
 $Comp
-L Connector:Conn_01x01_Male J5
+L Connector:Conn_01x01_Male J6
 U 1 1 5E6B2955
 P 3550 2150
-F 0 "J5" H 3522 2174 50  0000 R CNN
-F 1 "Reset Pad" H 3522 2083 50  0000 R CNN
+F 0 "J6" H 3522 2174 50  0000 R CNN
+F 1 "Reset" H 3522 2083 50  0000 R CNN
 F 2 "TestPoint:TestPoint_Pad_2.0x1.0mm" H 3550 2150 50  0001 C CNN
 F 3 "~" H 3550 2150 50  0001 C CNN
@@
 P 2250 1850
 F 0 "J1" H 2172 2467 50  0000 C CNN
-F 1 "Data Header" H 2172 2376 50  0000 C CNN
+F 1 "Peripherals" H 2172 2376 50  0000 C CNN
 F 2 "Connector_JST:JST_SH_BM09B-SRSS-TB_1x09-1MP_P1.00mm_Vertical" H 2250 1850 50  0001 C CNN
 F 3 "~" H 2250 1850 50  0001 C CNN
@@
 $EndComp
 $Comp
-L Connector:Conn_01x02_Male J2
+L Connector:Conn_01x02_Male J4
 U 1 1 5E6B02F6
 P 3550 1150
-F 0 "J2" H 3522 1124 50  0000 R CNN
-F 1 "USB Pads" H 3522 1033 50  0000 R CNN
+F 0 "J4" H 3522 1124 50  0000 R CNN
+F 1 "USB" H 3522 1033 50  0000 R CNN
 F 2 "TestPoint:TestPoint_2Pads_2.0x1.0mm" H 3550 1150 50  0001 C CNN
 F 3 "~" H 3550 1150 50  0001 C CNN
@@
 $EndComp
 $Comp
-L Connector:Conn_01x04_Male J4
+L Connector:Conn_01x04_Male J5
 U 1 1 5E6AE12F
 P 3550 1650
-F 0 "J4" H 3522 1624 50  0000 R CNN
-F 1 "GameCube Pads" H 3522 1533 50  0000 R CNN
+F 0 "J5" H 3522 1624 50  0000 R CNN
+F 1 "GameCube" H 3522 1533 50  0000 R CNN
 F 2 "TestPoint:TestPoint_4Pads_2.0x1.0mm" H 3550 1650 50  0001 C CNN
 F 3 "~" H 3550 1650 50  0001 C CNN
@@
 BT_D+
 $Comp
-L Connector_Generic_MountingPin:Conn_01x03_MountingPin J7
+L Connector_Generic_MountingPin:Conn_01x04_MountingPin J3
 U 1 1 5E6E5E9A
-P 2250 4200
-F 0 "J7" H 2172 4517 50  0000 C CNN
-F 1 "Video Header" H 2172 4426 50  0000 C CNN
-F 2 "Connector_JST:JST_SH_BM03B-SRSS-TB_1x03-1MP_P1.00mm_Vertical" H 2250 4200 50  0001 C CNN
-F 3 "~" H 2250 4200 50  0001 C CNN
-	1    2250 4200
-	-1   0    0    -1
-$EndComp
-$Comp
-L Connector_Generic_MountingPin:Conn_01x02_MountingPin J6
+P 2250 4350
+F 0 "J3" H 2172 4667 50  0000 C CNN
+F 1 "Video" H 2172 4576 50  0000 C CNN
+F 2 "Connector_JST:JST_SH_BM04B-SRSS-TB_1x04-1MP_P1.00mm_Vertical" H 2250 4350 50  0001 C CNN
+F 3 "~" H 2250 4350 50  0001 C CNN
+	1    2250 4350
+	-1   0    0    -1
+$EndComp
+$Comp
+L Connector:Conn_01x04_Male J9
+U 1 1 5E6E973B
+P 3550 4350
+F 0 "J9" H 3500 4300 50  0000 R CNN
+F 1 "Video" H 3500 4200 50  0000 R CNN
+F 2 "TestPoint:TestPoint_4Pads_2.0x1.0mm" H 3550 4350 50  0001 C CNN
+F 3 "~" H 3550 4350 50  0001 C CNN
+	1    3550 4350
+	-1   0    0    -1
+$EndComp
+$Comp
+L Connector:Conn_01x03_Male J8
+U 1 1 5E6EB339
+P 3550 3350
+F 0 "J8" H 3500 3350 50  0000 R CNN
+F 1 "Audio" H 3500 3250 50  0000 R CNN
+F 2 "TestPoint:TestPoint_3Pads_2.0x1.0mm" H 3550 3350 50  0001 C CNN
+F 3 "~" H 3550 3350 50  0001 C CNN
+	1    3550 3350
+	-1   0    0    -1
+$EndComp
+Wire Wire Line
+	2450 3250 3350 3250
+Wire Wire Line
+	2450 3350 3350 3350
+Wire Wire Line
+	2450 4250 3350 4250
+Wire Wire Line
+	2450 4350 3350 4350
+Wire Wire Line
+	2450 4450 3350 4450
+Text Label 3350 3250 2    50   ~ 0
+AUDIO_LEFT
+Text Label 3350 3350 2    50   ~ 0
+AUDIO_RIGHT
+Text Label 3350 4250 2    50   ~ 0
+VIDEO_Y
+Text Label 3350 4350 2    50   ~ 0
+VIDEO_PB
+Text Label 3350 4450 2    50   ~ 0
+VIDEO_PR
+$Comp
+L Mechanical:MountingHole_Pad H1
+U 1 1 5E6C8CF3
+P 750 1400
+F 0 "H1" H 850 1449 50  0000 L CNN
+F 1 "MountingHole_Pad" H 850 1358 50  0000 L CNN
+F 2 "MountingHole:MountingHole_2.7mm_M2.5_Pad_Via" H 750 1400 50  0001 C CNN
+F 3 "~" H 750 1400 50  0001 C CNN
+	1    750  1400
+	1    0    0    -1
+$EndComp
+$Comp
+L power:GND #PWR0101
+U 1 1 5E6C97A4
+P 750 1500
+F 0 "#PWR0101" H 750 1250 50  0001 C CNN
+F 1 "GND" H 755 1327 50  0000 C CNN
+F 2 "" H 750 1500 50  0001 C CNN
+F 3 "" H 750 1500 50  0001 C CNN
+	1    750  1500
+	1    0    0    -1
+$EndComp
+$Comp
+L Mechanical:MountingHole_Pad H2
+U 1 1 5E6CAB0C
+P 750 2000
+F 0 "H2" H 850 2049 50  0000 L CNN
+F 1 "MountingHole_Pad" H 850 1958 50  0000 L CNN
+F 2 "MountingHole:MountingHole_2.7mm_M2.5_Pad_Via" H 750 2000 50  0001 C CNN
+F 3 "~" H 750 2000 50  0001 C CNN
+	1    750  2000
+	1    0    0    -1
+$EndComp
+$Comp
+L power:GND #PWR0102
+U 1 1 5E6CAB12
+P 750 2100
+F 0 "#PWR0102" H 750 1850 50  0001 C CNN
+F 1 "GND" H 755 1927 50  0000 C CNN
+F 2 "" H 750 2100 50  0001 C CNN
+F 3 "" H 750 2100 50  0001 C CNN
+	1    750  2100
+	1    0    0    -1
+$EndComp
+$Comp
+L power:GND #PWR0106
+U 1 1 5E6D1C9C
+P 750 800
+F 0 "#PWR0106" H 750 550 50  0001 C CNN
+F 1 "GND" H 755 627 50  0000 C CNN
+F 2 "" H 750 800 50  0001 C CNN
+F 3 "" H 750 800 50  0001 C CNN
+	1    750  800
+	1    0    0    -1
+$EndComp
+$Comp
+L power:PWR_FLAG #FLG0101
+U 1 1 5E6D23F0
+P 750 800
+F 0 "#FLG0101" H 750 875 50  0001 C CNN
+F 1 "PWR_FLAG" H 750 973 50  0000 C CNN
+F 2 "" H 750 800 50  0001 C CNN
+F 3 "~" H 750 800 50  0001 C CNN
+	1    750  800
+	1    0    0    -1
+$EndComp
+$Comp
+L Connector_Generic_MountingPin:Conn_01x03_MountingPin J2
 U 1 1 5E6E7AC7
-P 2250 3200
-F 0 "J6" H 2172 3417 50  0000 C CNN
-F 1 "Audio Header" H 2172 3326 50  0000 C CNN
-F 2 "Connector_JST:JST_SH_BM02B-SRSS-TB_1x02-1MP_P1.00mm_Vertical" H 2250 3200 50  0001 C CNN
-F 3 "~" H 2250 3200 50  0001 C CNN
-	1    2250 3200
-	-1   0    0    -1
-$EndComp
-$Comp
-L Connector:Conn_01x03_Male J9
-U 1 1 5E6E973B
-P 3550 4200
-F 0 "J9" H 3522 4224 50  0000 R CNN
-F 1 "Video Pads" H 3522 4133 50  0000 R CNN
-F 2 "TestPoint:TestPoint_3Pads_2.0x1.0mm" H 3550 4200 50  0001 C CNN
-F 3 "~" H 3550 4200 50  0001 C CNN
-	1    3550 4200
-	-1   0    0    -1
-$EndComp
-$Comp
-L Connector:Conn_01x02_Male J8
-U 1 1 5E6EB339
-P 3550 3200
-F 0 "J8" H 3522 3174 50  0000 R CNN
-F 1 "Audio Pads" H 3522 3083 50  0000 R CNN
-F 2 "TestPoint:TestPoint_2Pads_2.0x1.0mm" H 3550 3200 50  0001 C CNN
-F 3 "~" H 3550 3200 50  0001 C CNN
-	1    3550 3200
-	-1   0    0    -1
-$EndComp
-Wire Wire Line
-	2450 3200 3350 3200
-Wire Wire Line
-	2450 3300 3350 3300
-Wire Wire Line
-	2450 4100 3350 4100
-Wire Wire Line
-	2450 4200 3350 4200
-Wire Wire Line
-	2450 4300 3350 4300
-Text Label 3350 3200 2    50   ~ 0
-AUDIO_LEFT
-Text Label 3350 3300 2    50   ~ 0
-AUDIO_RIGHT
-Text Label 3350 4100 2    50   ~ 0
-VIDEO_Y
-Text Label 3350 4200 2    50   ~ 0
-VIDEO_PB
-Text Label 3350 4300 2    50   ~ 0
-VIDEO_PR
+P 2250 3350
+F 0 "J2" H 2150 3700 50  0000 C CNN
+F 1 "Audio" H 2150 3600 50  0000 C CNN
+F 2 "Connector_JST:JST_SH_BM03B-SRSS-TB_1x03-1MP_P1.00mm_Vertical" H 2250 3350 50  0001 C CNN
+F 3 "~" H 2250 3350 50  0001 C CNN
+	1    2250 3350
+	-1   0    0    -1
+$EndComp
+Wire Wire Line
+	2450 3450 3350 3450
+Wire Wire Line
+	2450 4550 3350 4550
+Text Label 3350 3450 2    50   ~ 0
+AUDIO_GND
+Text Label 3350 4550 2    50   ~ 0
+VIDEO_GND
+NoConn ~ 2250 4750
+NoConn ~ 2250 2450
+NoConn ~ 2250 3650
 $EndSCHEMATC

Commit message: Shrink the board
Parts:
- J1: MPN (none) -> BM09B-SRSS-TB(LF)(SN); Manufacturer (none) -> JST
- J2: MPN (none) -> BM03B-SRSS-TB(LF)(SN); Manufacturer (none) -> JST
- J3: MPN (none) -> BM04B-SRSS-TB(LF)(SN); Manufacturer (none) -> JST
Changed lines of the file:
@@
 F 2 "Connector_JST:JST_SH_BM09B-SRSS-TB_1x09-1MP_P1.00mm_Vertical" H 2250 1850 50  0001 C CNN
 F 3 "~" H 2250 1850 50  0001 C CNN
+F 4 "JST" H 2250 1850 50  0001 C CNN "Manufacturer"
+F 5 "BM09B-SRSS-TB(LF)(SN)" H 2250 1850 50  0001 C CNN "MPN"
 	1    2250 1850
 	-1   0    0    -1
@@
 F 2 "Connector_JST:JST_SH_BM04B-SRSS-TB_1x04-1MP_P1.00mm_Vertical" H 2250 4350 50  0001 C CNN
 F 3 "~" H 2250 4350 50  0001 C CNN
+F 4 "JST" H 2250 4350 50  0001 C CNN "Manufacturer"
+F 5 "BM04B-SRSS-TB(LF)(SN)" H 2250 4350 50  0001 C CNN "MPN"
 	1    2250 4350
 	-1   0    0    -1
@@
 F 2 "Connector_JST:JST_SH_BM03B-SRSS-TB_1x03-1MP_P1.00mm_Vertical" H 2250 3350 50  0001 C CNN
 F 3 "~" H 2250 3350 50  0001 C CNN
+F 4 "JST" H 2250 3350 50  0001 C CNN "Manufacturer"
+F 5 "BM03B-SRSS-TB(LF)(SN)" H 2250 3350 50  0001 C CNN "MPN"
 	1    2250 3350
 	-1   0    0    -1

Commit message: v2.0
Parts:
- removed J8: Audio, TestPoint:TestPoint_3Pads_2.0x1.0mm, symbol Connector:Conn_01x03_Male
- added J10: Ground, project-footprints:TestPoint_Pad_2.0x1.0mm, symbol Connector:Conn_01x01_Male
- added J8: Audio, project-footprints:TestPoint_2Pads_2.0x1.0mm, symbol Connector:Conn_01x02_Male
- J4, J7: footprint TestPoint:TestPoint_2Pads_2.0x1.0mm -> project-footprints:TestPoint_2Pads_2.0x1.0mm
- J5: footprint TestPoint:TestPoint_4Pads_2.0x1.0mm -> project-footprints:TestPoint_4Pads_2.0x1.0mm
- J6: footprint TestPoint:TestPoint_Pad_2.0x1.0mm -> project-footprints:TestPoint_Pad_2.0x1.0mm
- J9: footprint TestPoint:TestPoint_4Pads_2.0x1.0mm -> project-footprints:TestPoint_3Pads_2.0x1.0mm; symbol Connector:Conn_01x04_Male -> Connector:Conn_01x03_Male
Connections:
- net AUDIO_GND is gone; now on net GND: J2.3 (Pin_3)
- net AUDIO_LEFT: now also J8.1 (Pin_1)
- net AUDIO_RIGHT: now also J8.2 (Pin_2)
- net GND: now also J3.4 (Pin_4), J10.1 (Pin_1)
- removed net VIDEO_GND: J3.4 (Pin_4), J9.4 (Pin_4)
Changed lines of the file:
@@
 F 0 "J7" H 3522 2424 50  0000 R CNN
 F 1 "Bluetooth" H 3522 2333 50  0000 R CNN
-F 2 "TestPoint:TestPoint_2Pads_2.0x1.0mm" H 3550 2450 50  0001 C CNN
+F 2 "project-footprints:TestPoint_2Pads_2.0x1.0mm" H 3550 2450 50  0001 C CNN
 F 3 "~" H 3550 2450 50  0001 C CNN
 	1    3550 2450
@@
 F 0 "J6" H 3522 2174 50  0000 R CNN
 F 1 "Reset" H 3522 2083 50  0000 R CNN
-F 2 "TestPoint:TestPoint_Pad_2.0x1.0mm" H 3550 2150 50  0001 C CNN
+F 2 "project-footprints:TestPoint_Pad_2.0x1.0mm" H 3550 2150 50  0001 C CNN
 F 3 "~" H 3550 2150 50  0001 C CNN
 	1    3550 2150
@@
 F 0 "J4" H 3522 1124 50  0000 R CNN
 F 1 "USB" H 3522 1033 50  0000 R CNN
-F 2 "TestPoint:TestPoint_2Pads_2.0x1.0mm" H 3550 1150 50  0001 C CNN
+F 2 "project-footprints:TestPoint_2Pads_2.0x1.0mm" H 3550 1150 50  0001 C CNN
 F 3 "~" H 3550 1150 50  0001 C CNN
 	1    3550 1150
@@
 F 0 "J5" H 3522 1624 50  0000 R CNN
 F 1 "GameCube" H 3522 1533 50  0000 R CNN
-F 2 "TestPoint:TestPoint_4Pads_2.0x1.0mm" H 3550 1650 50  0001 C CNN
+F 2 "project-footprints:TestPoint_4Pads_2.0x1.0mm" H 3550 1650 50  0001 C CNN
 F 3 "~" H 3550 1650 50  0001 C CNN
 	1    3550 1650
@@
 	-1   0    0    -1
 $EndComp
-$Comp
-L Connector:Conn_01x04_Male J9
-U 1 1 5E6E973B
-P 3550 4350
-F 0 "J9" H 3500 4300 50  0000 R CNN
-F 1 "Video" H 3500 4200 50  0000 R CNN
-F 2 "TestPoint:TestPoint_4Pads_2.0x1.0mm" H 3550 4350 50  0001 C CNN
-F 3 "~" H 3550 4350 50  0001 C CNN
-	1    3550 4350
-	-1   0    0    -1
-$EndComp
-$Comp
-L Connector:Conn_01x03_Male J8
-U 1 1 5E6EB339
-P 3550 3350
-F 0 "J8" H 3500 3350 50  0000 R CNN
-F 1 "Audio" H 3500 3250 50  0000 R CNN
-F 2 "TestPoint:TestPoint_3Pads_2.0x1.0mm" H 3550 3350 50  0001 C CNN
-F 3 "~" H 3550 3350 50  0001 C CNN
-	1    3550 3350
-	-1   0    0    -1
-$EndComp
 Wire Wire Line
 	2450 3250 3350 3250
@@
 	1    0    0    -1
 $EndComp
+NoConn ~ 2250 4750
+NoConn ~ 2250 2450
+$Comp
+L Connector:Conn_01x01_Male J10
+U 1 1 5E825F7C
+P 3550 5050
+F 0 "J10" H 3522 5074 50  0000 R CNN
+F 1 "Ground" H 3522 4983 50  0000 R CNN
+F 2 "project-footprints:TestPoint_Pad_2.0x1.0mm" H 3550 5050 50  0001 C CNN
+F 3 "~" H 3550 5050 50  0001 C CNN
+	1    3550 5050
+	-1   0    0    -1
+$EndComp
+$Comp
+L power:GND #PWR0103
+U 1 1 5E827D09
+P 2550 5150
+F 0 "#PWR0103" H 2550 4900 50  0001 C CNN
+F 1 "GND" H 2555 4977 50  0000 C CNN
+F 2 "" H 2550 5150 50  0001 C CNN
+F 3 "" H 2550 5150 50  0001 C CNN
+	1    2550 5150
+	1    0    0    -1
+$EndComp
+NoConn ~ 2250 3650
 $Comp
 L Connector_Generic_MountingPin:Conn_01x03_MountingPin J2
@@
 	-1   0    0    -1
 $EndComp
-Wire Wire Line
-	2450 3450 3350 3450
-Wire Wire Line
-	2450 4550 3350 4550
-Text Label 3350 3450 2    50   ~ 0
-AUDIO_GND
-Text Label 3350 4550 2    50   ~ 0
-VIDEO_GND
-NoConn ~ 2250 4750
-NoConn ~ 2250 2450
-NoConn ~ 2250 3650
+$Comp
+L power:GND #PWR0104
+U 1 1 5E82BC0E
+P 2550 3500
+F 0 "#PWR0104" H 2550 3250 50  0001 C CNN
+F 1 "GND" H 2555 3327 50  0000 C CNN
+F 2 "" H 2550 3500 50  0001 C CNN
+F 3 "" H 2550 3500 50  0001 C CNN
+	1    2550 3500
+	1    0    0    -1
+$EndComp
+Wire Wire Line
+	2450 3450 2550 3450
+Wire Wire Line
+	2550 3450 2550 3500
+$Comp
+L Connector:Conn_01x03_Male J9
+U 1 1 5E6E973B
+P 3550 4350
+F 0 "J9" H 3500 4300 50  0000 R CNN
+F 1 "Video" H 3500 4200 50  0000 R CNN
+F 2 "project-footprints:TestPoint_3Pads_2.0x1.0mm" H 3550 4350 50  0001 C CNN
+F 3 "~" H 3550 4350 50  0001 C CNN
+	1    3550 4350
+	-1   0    0    -1
+$EndComp
+$Comp
+L power:GND #PWR0105
+U 1 1 5E82EE8D
+P 2550 4600
+F 0 "#PWR0105" H 2550 4350 50  0001 C CNN
+F 1 "GND" H 2555 4427 50  0000 C CNN
+F 2 "" H 2550 4600 50  0001 C CNN
+F 3 "" H 2550 4600 50  0001 C CNN
+	1    2550 4600
+	1    0    0    -1
+$EndComp
+Wire Wire Line
+	2450 4550 2550 4550
+Wire Wire Line
+	2550 4550 2550 4600
+Wire Wire Line
+	3350 5050 2550 5050
+Wire Wire Line
+	2550 5050 2550 5150
+$Comp
+L Connector:Conn_01x02_Male J8
+U 1 1 5E834D7E
+P 3550 3250
+F 0 "J8" H 3500 3200 50  0000 R CNN
+F 1 "Audio" H 3500 3100 50  0000 R CNN
+F 2 "project-footprints:TestPoint_2Pads_2.0x1.0mm" H 3550 3250 50  0001 C CNN
+F 3 "~" H 3550 3250 50  0001 C CNN
+	1    3550 3250
+	-1   0    0    -1
+$EndComp
 $EndSCHEMATC

Commit message: v3.0 - minimal size, cutout for mobo cap, split USB from data header, reorder GC lines to match mobo
Parts:
- removed J10: Ground, project-footprints:TestPoint_Pad_2.0x1.0mm, symbol Connector:Conn_01x01_Male
- added J10: USB, Connector_JST:JST_SH_BM02B-SRSS-TB_1x02-1MP_P1.00mm_Vertical, symbol Connector_Generic:Conn_01x02
- H1, H2: footprint MountingHole:MountingHole_2.7mm_M2.5_Pad_Via -> MountingHole:MountingHole_2.7mm_M2.5_ISO14580_Pad
- J1: footprint Connector_JST:JST_SH_BM09B-SRSS-TB_1x09-1MP_P1.00mm_Vertical -> Connector_JST:JST_SH_BM07B-SRSS-TB_1x07-1MP_P1.00mm_Vertical; symbol Connector_Generic_MountingPin:Conn_01x09_MountingPin -> Connector_Generic:Conn_01x07
- J2: symbol Connector_Generic_MountingPin:Conn_01x03_MountingPin -> Connector_Generic:Conn_01x03
- J3: symbol Connector_Generic_MountingPin:Conn_01x04_MountingPin -> Connector_Generic:Conn_01x04
- J5: value GameCube -> GC
- J6: value Reset -> RST
- J7: value Bluetooth -> BT
Connections:
- net AUDIO_LEFT: now also J2.3 (Pin_3); no longer J2.1 (Pin_1)
- net BT_D+: now also J1.2 (Pin_2), J7.2 (Pin_2); no longer J1.8 (Pin_8), J7.1 (Pin_1)
- net BT_D-: now also J1.1 (Pin_1), J7.1 (Pin_1); no longer J1.9 (Pin_9), J7.2 (Pin_2)
- net GC_1: now also J1.4 (Pin_4), J5.2 (Pin_2); no longer J1.6 (Pin_6), J5.4 (Pin_4)
- net GC_2: now also J5.1 (Pin_1); no longer J5.3 (Pin_3)
- net GC_3: now also J1.6 (Pin_6), J5.3 (Pin_3); no longer J1.4 (Pin_4), J5.2 (Pin_2)
- net GC_4: now also J1.7 (Pin_7), J5.4 (Pin_4); no longer J1.3 (Pin_3), J5.1 (Pin_1)
- net GND: now also J2.1 (Pin_1), J3.1 (Pin_1); no longer J2.3 (Pin_3), J3.4 (Pin_4)
- net RST: now also J1.3 (Pin_3); no longer J1.7 (Pin_7)
- net USB_D+: now also J4.2 (Pin_2), J10.1 (Pin_1); no longer J1.1 (Pin_1), J4.1 (Pin_1)
- net USB_D-: now also J4.1 (Pin_1), J10.2 (Pin_2); no longer J1.2 (Pin_2), J4.2 (Pin_2)
- net VIDEO_PB: now also J3.3 (Pin_3); no longer J3.2 (Pin_2)
- net VIDEO_PR: now also J3.2 (Pin_2); no longer J3.3 (Pin_3)
- net VIDEO_Y: now also J3.4 (Pin_4); no longer J3.1 (Pin_1)
- no-connect marks 3 -> 0
Other:
- moved on the sheet: J4, J5, J6
